File: pcb/main-trackball/main.kicad_pcb (KiCad board)
At the start: 2 copper layers, 174 x 111.8 mm, 78 parts, among them J1 Conn_01x04, J10 JTAG, J2 USB_B, J3 Trackball_conn, J4 ROW0, J5 RJ45, J6 ROW1, J7 ROW2, J8 ROW3, J9 STLink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

Commit message: wiring
Parts:
- removed the REF** at (263.5, 147.3)
- removed the REF** at (263.5, 128.3)
- added REF**: MountingHole_3.2mm_M3, MountingHole:MountingHole_3.2mm_M3, F.Cu at (161.9, 62.2)
- added REF**: MountingHole_3.2mm_M3, MountingHole:MountingHole_3.2mm_M3, F.Cu at (161.9, 43.2)
- moved C1 132.5 mm to (22.6, 68.2)
- moved C10 132.5 mm to (10.7, 38.4)
- moved C11 132.5 mm to (25.1, 38.5)
- moved C2 132.5 mm to (25.1, 69.8)
- moved C3 132.5 mm to (7.37, 39.5)
- moved C4 132.5 mm to (7.37, 41.0)
- moved C5 132.5 mm to (6.35, 43.6)
- moved C6 132.5 mm to (11.9, 49.1)
- moved C9 132.5 mm to (18.0, 31.4)
- moved D4 132.5 mm to (73.0, 73.7)
- moved D5 132.5 mm to (3.17, 20.3)
- moved D6 132.5 mm to (3.17, 17.8)
- moved D7 132.5 mm to (3.17, 15.2)
- moved G*** 132.5 mm to (87.6, 39.4) (x2)
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Routing:
- net /SELECT4: track 0.00 -> 162.3 mm, vias 0 -> 1
- net +5V: track 8.31 -> 142.1 mm, vias 1 -> 7
- net +3V3: track 224.1 -> 312.6 mm, vias 11 -> 12
- net /SCK: track 42.5 -> 91.9 mm, vias 1 -> 2
- net /MISO: track 40.3 -> 87.9 mm
- net /MOSI: track 42.8 -> 79.8 mm, vias 1 -> 2
- net Net-(D1-Pad1): track 0.00 -> 34.3 mm
- net /SS_K: track 5.49 -> 36.3 mm, vias 0 -> 5
- net /SS_T: track 41.7 -> 70.9 mm
- net Net-(D4-Pad1): track 0.00 -> 25.9 mm, vias 0 -> 1
- net GND: track 342.0 -> 358.3 mm, vias 10 -> 11
- net /READ3: track 241.7 -> 247.4 mm, vias 3 -> 4
- net /READ1: track 232.5 -> 229.6 mm
Other:
- net class Default: trace_width 0.25 -> 0.127; via_dia 0.8 -> 0.5; via_drill 0.4 -> 0.2
- rule trace_min: 0 -> 0.127
- rule via_min_drill: 0.3 -> 0.2
- rule via_min_size: 0.4 -> 0.45
