File: pcb/row/row.kicad_pcb (KiCad board)
At the start: 2 copper layers, 138.4 x 17.8 mm, 15 parts, among them J1 INTERFACE, SW1 SW0, SW2 SW1, SW3 SW2, SW4 SW3, SW5 SW4, SW6 SW5

Commit message: fix design
Parts:
- added REF**: MountingHole_2.2mm_M2, MountingHole:MountingHole_2.2mm_M2, F.Cu at (24.8, 6.35)
- added REF**: MountingHole_2.2mm_M2, MountingHole:MountingHole_2.2mm_M2, F.Cu at (81.9, -6.35)
- added REF**: MountingHole_2.2mm_M2, MountingHole:MountingHole_2.2mm_M2, F.Cu at (81.9, 6.35)
- added REF**: MountingHole_2.2mm_M2, MountingHole:MountingHole_2.2mm_M2, F.Cu at (101.0, 6.35)
- added REF**: MountingHole_2.2mm_M2, MountingHole:MountingHole_2.2mm_M2, F.Cu at (101.0, -6.35)
- added REF**: MountingHole_2.2mm_M2, MountingHole:MountingHole_2.2mm_M2, F.Cu at (62.9, -6.35)
- added REF**: MountingHole_2.2mm_M2, MountingHole:MountingHole_2.2mm_M2, F.Cu at (62.9, 6.35)
- added REF**: MountingHole_2.2mm_M2, MountingHole:MountingHole_2.2mm_M2, F.Cu at (43.8, -6.35)
- added REF**: MountingHole_2.2mm_M2, MountingHole:MountingHole_2.2mm_M2, F.Cu at (43.8, 6.35)
- added REF**: MountingHole_2.2mm_M2, MountingHole:MountingHole_2.2mm_M2, F.Cu at (24.8, -6.35)
- moved D6 126.0 mm to (101.0, 0.00)
- moved D5 125.3 mm to (81.9, 0.00)
- moved D1 124.5 mm to (5.71, 0.00)
- moved SW6 124.0 mm to (110.5, 3.81)
- moved D2 123.8 mm to (24.8, 0.00)
- moved J1 123.3 mm to (123.2, 7.62)
- moved REF** 123.3 mm to (0.00, 0.00)
- moved REF** 123.3 mm to (130.8, 0.00)
- moved SW2 123.3 mm to (34.3, 1.27)
- moved SW3 123.3 mm to (53.3, -1.27)
- moved SW5 123.3 mm to (91.4, 3.81)
- moved SW1 123.3 mm to (15.2, 2.54)
- moved SW4 123.3 mm to (72.4, 0.00)
- moved D4 123.1 mm to (62.9, 0.00)
- moved D3 122.4 mm to (43.8, 0.00)
Routing:
- net /READ1: track 110.4 -> 102.2 mm, vias 0 -> 1
- net /SELECT: track 144.4 -> 152.4 mm
- net Net-(D6-Pad1): track 29.5 -> 21.6 mm
- net Net-(D2-Pad1): track 29.5 -> 21.9 mm
- net Net-(D4-Pad1): track 29.5 -> 22.0 mm
- net Net-(D5-Pad1): track 28.9 -> 22.1 mm
- net Net-(D1-Pad1): track 27.3 -> 21.6 mm
- net /READ2: track 89.2 -> 83.8 mm, vias 0 -> 1
- net /READ5: track 26.9 -> 31.6 mm, vias 1 -> 0
- net /READ4: track 47.9 -> 50.3 mm, vias 1 -> 0
- net /READ0: track 119.3 -> 121.4 mm, vias 0 -> 1
- net Net-(D3-Pad1): track 29.1 -> 28.3 mm
- net /READ3: track 66.9 -> 66.4 mm, vias 1 -> 0
