File: pcb/trackball/trackball.sch (KiCad schematic (older format))
At the start: 23 parts, among them SW1 BTN, U1 AN48841B, U2 AN48841B, U3 AN48841B, U4 AN48841B

Commit message: complete trackball breakout
Parts:
- removed D1, D2, D3, D4: LED, LED_SMD:LED_0201_0603Metric, symbol Device:LED
- removed R1, R2, R4, R5: R, Resistor_SMD:R_0201_0603Metric, symbol Device:R
- added J1, J2, J3, J4, J5, J6, J7: Conn_01x01_Female, TestPoint:TestPoint_THTPad_D1.0mm_Drill0.5mm, symbol Connector:Conn_01x01_Female
- R3, R6, R7, R8, R9: footprint Resistor_SMD:R_0201_0603Metric -> Resistor_SMD:R_0603_1608Metric
- SW1: footprint (none) -> folivora:Film_Switch_4X4X0.8MM
- U1, U2, U3, U4: symbol folivora:AN48841B -> trackball-rescue:AN48841B-folivora
Connections:
- net labels removed: LED1, LED2, LED3, LED4
- wire segments 56 -> 52
Changed lines of the file:
@@
 EESchema Schematic File Version 4
+LIBS:trackball-cache
 EELAYER 29 0
 EELAYER END
@@
 $EndDescr
 $Comp
-L folivora:AN48841B U1
+L trackball-rescue:AN48841B-folivora U1
 U 1 1 5D35C0DC
 P 2900 3100
@@
 F 0 "R6" H 3470 2896 50  0000 L CNN
 F 1 "10k" H 3470 2805 50  0000 L CNN
-F 2 "Resistor_SMD:R_0201_0603Metric" V 3330 2850 50  0001 C CNN
+F 2 "Resistor_SMD:R_0603_1608Metric" V 3330 2850 50  0001 C CNN
 F 3 "~" H 3400 2850 50  0001 C CNN
 	1    3400 2850
@@
 	3400 3100 3300 3100
 $Comp
-L folivora:AN48841B U2
+L trackball-rescue:AN48841B-folivora U2
 U 1 1 5D35D74C
 P 2900 3850
@@
 F 0 "R7" H 3470 3646 50  0000 L CNN
 F 1 "10k" H 3470 3555 50  0000 L CNN
-F 2 "Resistor_SMD:R_0201_0603Metric" V 3330 3600 50  0001 C CNN
+F 2 "Resistor_SMD:R_0603_1608Metric" V 3330 3600 50  0001 C CNN
 F 3 "~" H 3400 3600 50  0001 C CNN
 	1    3400 3600
@@
 	3400 3850 3300 3850
 $Comp
-L folivora:AN48841B U3
+L trackball-rescue:AN48841B-folivora U3
 U 1 1 5D35E7FC
 P 2900 4600
@@
 F 0 "R8" H 3470 4396 50  0000 L CNN
 F 1 "10k" H 3470 4305 50  0000 L CNN
-F 2 "Resistor_SMD:R_0201_0603Metric" V 3330 4350 50  0001 C CNN
+F 2 "Resistor_SMD:R_0603_1608Metric" V 3330 4350 50  0001 C CNN
 F 3 "~" H 3400 4350 50  0001 C CNN
 	1    3400 4350
@@
 	3400 4600 3300 4600
 $Comp
-L folivora:AN48841B U4
+L trackball-rescue:AN48841B-folivora U4
 U 1 1 5D35E81D
 P 2900 5350
@@
 F 0 "R9" H 3470 5146 50  0000 L CNN
 F 1 "10k" H 3470 5055 50  0000 L CNN
-F 2 "Resistor_SMD:R_0201_0603Metric" V 3330 5100 50  0001 C CNN
+F 2 "Resistor_SMD:R_0603_1608Metric" V 3330 5100 50  0001 C CNN
 F 3 "~" H 3400 5100 50  0001 C CNN
 	1    3400 5100
@@
 	800  3850 800  3750
 $Comp
-L Device:LED D4
-U 1 1 5D36E81F
-P 1550 5300
-F 0 "D4" H 1750 5350 50  0000 R CNN
-F 1 "LED" H 1450 5350 50  0000 R CNN
-F 2 "LED_SMD:LED_0201_0603Metric" H 1550 5300 50  0001 C CNN
-F 3 "~" H 1550 5300 50  0001 C CNN
-	1    1550 5300
-	0    -1   -1   0
-$EndComp
-$Comp
-L Device:R R5
-U 1 1 5D36F1FB
-P 1550 4900
-F 0 "R5" H 1620 4946 50  0000 L CNN
-F 1 "R" H 1620 4855 50  0000 L CNN
-F 2 "Resistor_SMD:R_0201_0603Metric" V 1480 4900 50  0001 C CNN
-F 3 "~" H 1550 4900 50  0001 C CNN
-	1    1550 4900
-	1    0    0    -1
-$EndComp
-$Comp
-L power:GND #PWR0115
-U 1 1 5D36FB13
-P 1550 5550
-F 0 "#PWR0115" H 1550 5300 50  0001 C CNN
-F 1 "GND" H 1555 5377 50  0000 C CNN
-F 2 "" H 1550 5550 50  0001 C CNN
-F 3 "" H 1550 5550 50  0001 C CNN
-	1    1550 5550
-	1    0    0    -1
-$EndComp
-Wire Wire Line
-	1550 5550 1550 5450
-Wire Wire Line
-	1550 5150 1550 5050
-$Comp
-L Device:LED D3
-U 1 1 5D372A6A
-P 1300 5300
-F 0 "D3" H 1500 5350 50  0000 R CNN
-F 1 "LED" H 1200 5350 50  0000 R CNN
-F 2 "LED_SMD:LED_0201_0603Metric" H 1300 5300 50  0001 C CNN
-F 3 "~" H 1300 5300 50  0001 C CNN
-	1    1300 5300
-	0    -1   -1   0
-$EndComp
-$Comp
-L Device:R R4
-U 1 1 5D372A74
-P 1300 4900
-F 0 "R4" H 1370 4946 50  0000 L CNN
-F 1 "R" H 1370 4855 50  0000 L CNN
-F 2 "Resistor_SMD:R_0201_0603Metric" V 1230 4900 50  0001 C CNN
-F 3 "~" H 1300 4900 50  0001 C CNN
-	1    1300 4900
-	1    0    0    -1
-$EndComp
-$Comp
-L power:GND #PWR0116
-U 1 1 5D372A7E
-P 1300 5550
-F 0 "#PWR0116" H 1300 5300 50  0001 C CNN
-F 1 "GND" H 1305 5377 50  0000 C CNN
-F 2 "" H 1300 5550 50  0001 C CNN
-F 3 "" H 1300 5550 50  0001 C CNN
-	1    1300 5550
-	1    0    0    -1
-$EndComp
-Wire Wire Line
-	1300 5550 1300 5450
-Wire Wire Line
-	1300 5150 1300 5050
-$Comp
-L Device:LED D2
-U 1 1 5D377C27
-P 1050 5300
-F 0 "D2" H 1250 5350 50  0000 R CNN
-F 1 "LED" H 950 5350 50  0000 R CNN
-F 2 "LED_SMD:LED_0201_0603Metric" H 1050 5300 50  0001 C CNN
-F 3 "~" H 1050 5300 50  0001 C CNN
-	1    1050 5300
-	0    -1   -1   0
-$EndComp
-$Comp
-L Device:R R2
-U 1 1 5D377C31
-P 1050 4900
-F 0 "R2" H 1120 4946 50  0000 L CNN
-F 1 "R" H 1120 4855 50  0000 L CNN
-F 2 "Resistor_SMD:R_0201_0603Metric" V 980 4900 50  0001 C CNN
-F 3 "~" H 1050 4900 50  0001 C CNN
-	1    1050 4900
-	1    0    0    -1
-$EndComp
-$Comp
-L power:GND #PWR0117
-U 1 1 5D377C3B
-P 1050 5550
-F 0 "#PWR0117" H 1050 5300 50  0001 C CNN
-F 1 "GND" H 1055 5377 50  0000 C CNN
-F 2 "" H 1050 5550 50  0001 C CNN
-F 3 "" H 1050 5550 50  0001 C CNN
-	1    1050 5550
-	1    0    0    -1
-$EndComp
-Wire Wire Line
-	1050 5550 1050 5450
-Wire Wire Line
-	1050 5150 1050 5050
-$Comp
-L Device:LED D1
-U 1 1 5D377C47
-P 800 5300
-F 0 "D1" H 1000 5350 50  0000 R CNN
-F 1 "LED" H 700 5350 50  0000 R CNN
-F 2 "LED_SMD:LED_0201_0603Metric" H 800 5300 50  0001 C CNN
-F 3 "~" H 800 5300 50  0001 C CNN
-	1    800  5300
-	0    -1   -1   0
-$EndComp
-$Comp
-L Device:R R1
-U 1 1 5D377C51
-P 800 4900
-F 0 "R1" H 870 4946 50  0000 L CNN
-F 1 "R" H 870 4855 50  0000 L CNN
-F 2 "Resistor_SMD:R_0201_0603Metric" V 730 4900 50  0001 C CNN
-F 3 "~" H 800 4900 50  0001 C CNN
-	1    800  4900
-	1    0    0    -1
-$EndComp
-$Comp
-L power:GND #PWR0118
-U 1 1 5D377C5B
-P 800 5550
-F 0 "#PWR0118" H 800 5300 50  0001 C CNN
-F 1 "GND" H 805 5377 50  0000 C CNN
-F 2 "" H 800 5550 50  0001 C CNN
-F 3 "" H 800 5550 50  0001 C CNN
-	1    800  5550
-	1    0    0    -1
-$EndComp
-Wire Wire Line
-	800  5550 800  5450
-Wire Wire Line
-	800  5150 800  5050
-Text Label 800  4750 0    50   ~ 0
-LED1
-Text Label 1050 4750 0    50   ~ 0
-LED2
-Text Label 1300 4750 0    50   ~ 0
-LED3
-Text Label 1550 4750 0    50   ~ 0
-LED4
-$Comp
 L Switch:SW_DPST SW1
 U 1 1 5D38C32C
@@
 F 0 "SW1" H 1550 2875 50  0000 C CNN
 F 1 "BTN" H 1550 2784 50  0000 C CNN
-F 2 "" H 1550 2550 50  0001 C CNN
+F 2 "folivora:Film_Switch_4X4X0.8MM" H 1550 2550 50  0001 C CNN
 F 3 "~" H 1550 2550 50  0001 C CNN
 	1    1550 2550
@@
 F 0 "R3" V 1150 2300 50  0000 L CNN
 F 1 "10k" V 1150 2100 50  0000 L CNN
-F 2 "Resistor_SMD:R_0201_0603Metric" V 1180 2200 50  0001 C CNN
+F 2 "Resistor_SMD:R_0603_1608Metric" V 1180 2200 50  0001 C CNN
 F 3 "~" H 1250 2200 50  0001 C CNN
 	1    1250 2200
@@
 Text Label 3400 5350 0    50   ~ 0
 LEFT
+$Comp
+L Connector:Conn_01x01_Female J1
+U 1 1 5D383FC3
+P 4600 3200
+F 0 "J1" H 4628 3226 50  0000 L CNN
+F 1 "Conn_01x01_Female" H 4628 3135 50  0000 L CNN
+F 2 "TestPoint:TestPoint_THTPad_D1.0mm_Drill0.5mm" H 4600 3200 50  0001 C CNN
+F 3 "~" H 4600 3200 50  0001 C CNN
+	1    4600 3200
+	1    0    0    -1
+$EndComp
+$Comp
+L power:+5V #PWR0115
+U 1 1 5D38474E
+P 4300 3100
+F 0 "#PWR0115" H 4300 2950 50  0001 C CNN
+F 1 "+5V" H 4315 3273 50  0000 C CNN
+F 2 "" H 4300 3100 50  0001 C CNN
+F 3 "" H 4300 3100 50  0001 C CNN
+	1    4300 3100
+	1    0    0    -1
+$EndComp
+Wire Wire Line
+	4300 3100 4300 3200
+Wire Wire Line
+	4300 3200 4400 3200
+$Comp
+L power:GND #PWR0116
+U 1 1 5D38663C
+P 4300 4200
+F 0 "#PWR0116" H 4300 3950 50  0001 C CNN
+F 1 "GND" H 4305 4027 50  0000 C CNN
+F 2 "" H 4300 4200 50  0001 C CNN
+F 3 "" H 4300 4200 50  0001 C CNN
+	1    4300 4200
+	1    0    0    -1
+$EndComp
+$Comp
+L Connector:Conn_01x01_Female J7
+U 1 1 5D386BCE
+P 4600 4100
+F 0 "J7" H 4628 4126 50  0000 L CNN
+F 1 "Conn_01x01_Female" H 4628 4035 50  0000 L CNN
+F 2 "TestPoint:TestPoint_THTPad_D1.0mm_Drill0.5mm" H 4600 4100 50  0001 C CNN
+F 3 "~" H 4600 4100 50  0001 C CNN
+	1    4600 4100
+	1    0    0    -1
+$EndComp
+Wire Wire Line
+	4300 4200 4300 4100
+Wire Wire Line
+	4300 4100 4400 4100
+$Comp
+L Connector:Conn_01x01_Female J2
+U 1 1 5D38B195
+P 4600 3350
+F 0 "J2" H 4628 3376 50  0000 L CNN
+F 1 "Conn_01x01_Female" H 4628 3285 50  0000 L CNN
+F 2 "TestPoint:TestPoint_THTPad_D1.0mm_Drill0.5mm" H 4600 3350 50  0001 C CNN
+F 3 "~" H 4600 3350 50  0001 C CNN
+	1    4600 3350
+	1    0    0    -1
+$EndComp
+$Comp
+L Connector:Conn_01x01_Female J3
+U 1 1 5D38BA78
+P 4600 3500
+F 0 "J3" H 4628 3526 50  0000 L CNN
+F 1 "Conn_01x01_Female" H 4628 3435 50  0000 L CNN
+F 2 "TestPoint:TestPoint_THTPad_D1.0mm_Drill0.5mm" H 4600 3500 50  0001 C CNN
+F 3 "~" H 4600 3500 50  0001 C CNN
+	1    4600 3500
+	1    0    0    -1
+$EndComp
+$Comp
+L Connector:Conn_01x01_Female J4
+U 1 1 5D38C1BA
+P 4600 3650
+F 0 "J4" H 4628 3676 50  0000 L CNN
+F 1 "Conn_01x01_Female" H 4628 3585 50  0000 L CNN
+F 2 "TestPoint:TestPoint_THTPad_D1.0mm_Drill0.5mm" H 4600 3650 50  0001 C CNN
+F 3 "~" H 4600 3650 50  0001 C CNN
+	1    4600 3650
+	1    0    0    -1
+$EndComp
+$Comp
+L Connector:Conn_01x01_Female J5
+U 1 1 5D38C1C4
+P 4600 3800
+F 0 "J5" H 4628 3826 50  0000 L CNN
+F 1 "Conn_01x01_Female" H 4628 3735 50  0000 L CNN
+F 2 "TestPoint:TestPoint_THTPad_D1.0mm_Drill0.5mm" H 4600 3800 50  0001 C CNN
+F 3 "~" H 4600 3800 50  0001 C CNN
+	1    4600 3800
+	1    0    0    -1
+$EndComp
+$Comp
+L Connector:Conn_01x01_Female J6
+U 1 1 5D38DA7A
+P 4600 3950
+F 0 "J6" H 4628 3976 50  0000 L CNN
+F 1 "Conn_01x01_Female" H 4628 3885 50  0000 L CNN
+F 2 "TestPoint:TestPoint_THTPad_D1.0mm_Drill0.5mm" H 4600 3950 50  0001 C CNN
+F 3 "~" H 4600 3950 50  0001 C CNN
+	1    4600 3950
+	1    0    0    -1
+$EndComp
+Text Label 4400 3350 2    50   ~ 0
+UP
+Text Label 4400 3500 2    50   ~ 0
+RIGHT
+Text Label 4400 3800 2    50   ~ 0
+LEFT
+Text Label 4400 3650 2    50   ~ 0
+DOWN
+Text Label 4400 3950 2    50   ~ 0
+BTN
 $EndSCHEMATC

Commit message: trackball breakout
Parts:
- removed C2: 1uF, Capacitor_SMD:C_0805_2012Metric, symbol Device:C
- removed J6: Conn_01x01_Female, TestPoint:TestPoint_THTPad_D1.0mm_Drill0.5mm, symbol Connector:Conn_01x01_Female
- removed R3: 10k, Resistor_SMD:R_0603_1608Metric, symbol Device:R
- removed SW1: BTN, folivora:Film_Switch_4X4X0.8MM, symbol Switch:SW_DPST
- J1: value Conn_01x01_Female -> 5V
- J2: value Conn_01x01_Female -> UP
- J3: value Conn_01x01_Female -> R
- J4: value Conn_01x01_Female -> D
- J5: value Conn_01x01_Female -> L
- J7: value Conn_01x01_Female -> GND
- U1, U2, U3, U4: footprint folivora:SMINI-5DE -> folivora:SMINI_5DE
Connections:
- net labels removed: BTN
- wire segments 52 -> 40
Changed lines of the file:
@@
 F 0 "U1" H 2900 3425 50  0000 C CNN
 F 1 "AN48841B" H 2900 3334 50  0000 C CNN
-F 2 "folivora:SMINI-5DE" H 2600 2850 50  0001 C CNN
+F 2 "folivora:SMINI_5DE" H 2600 2850 50  0001 C CNN
 F 3 "" H 2600 2850 50  0001 C CNN
 	1    2900 3100
@@
 F 0 "U2" H 2900 4175 50  0000 C CNN
 F 1 "AN48841B" H 2900 4084 50  0000 C CNN
-F 2 "folivora:SMINI-5DE" H 2600 3600 50  0001 C CNN
+F 2 "folivora:SMINI_5DE" H 2600 3600 50  0001 C CNN
 F 3 "" H 2600 3600 50  0001 C CNN
 	1    2900 3850
@@
 F 0 "U3" H 2900 4925 50  0000 C CNN
 F 1 "AN48841B" H 2900 4834 50  0000 C CNN
-F 2 "folivora:SMINI-5DE" H 2600 4350 50  0001 C CNN
+F 2 "folivora:SMINI_5DE" H 2600 4350 50  0001 C CNN
 F 3 "" H 2600 4350 50  0001 C CNN
 	1    2900 4600
@@
 F 0 "U4" H 2900 5675 50  0000 C CNN
 F 1 "AN48841B" H 2900 5584 50  0000 C CNN
-F 2 "folivora:SMINI-5DE" H 2600 5100 50  0001 C CNN
+F 2 "folivora:SMINI_5DE" H 2600 5100 50  0001 C CNN
 F 3 "" H 2600 5100 50  0001 C CNN
 	1    2900 5350
@@
 Wire Wire Line
 	800  3850 800  3750
-$Comp
-L Switch:SW_DPST SW1
-U 1 1 5D38C32C
-P 1550 2550
-F 0 "SW1" H 1550 2875 50  0000 C CNN
-F 1 "BTN" H 1550 2784 50  0000 C CNN
-F 2 "folivora:Film_Switch_4X4X0.8MM" H 1550 2550 50  0001 C CNN
-F 3 "~" H 1550 2550 50  0001 C CNN
-	1    1550 2550
-	1    0    0    -1
-$EndComp
-$Comp
-L Device:R R3
-U 1 1 5D38D89E
-P 1250 2200
-F 0 "R3" V 1150 2300 50  0000 L CNN
-F 1 "10k" V 1150 2100 50  0000 L CNN
-F 2 "Resistor_SMD:R_0603_1608Metric" V 1180 2200 50  0001 C CNN
-F 3 "~" H 1250 2200 50  0001 C CNN
-	1    1250 2200
-	1    0    0    -1
-$EndComp
-$Comp
-L Device:C C2
-U 1 1 5D38E42F
-P 1000 2650
-F 0 "C2" V 748 2650 50  0000 C CNN
-F 1 "1uF" V 839 2650 50  0000 C CNN
-F 2 "Capacitor_SMD:C_0805_2012Metric" H 1038 2500 50  0001 C CNN
-F 3 "~" H 1000 2650 50  0001 C CNN
-	1    1000 2650
-	0    1    1    0
-$EndComp
-$Comp
-L power:GND #PWR0119
-U 1 1 5D38F375
-P 750 2750
-F 0 "#PWR0119" H 750 2500 50  0001 C CNN
-F 1 "GND" H 755 2577 50  0000 C CNN
-F 2 "" H 750 2750 50  0001 C CNN
-F 3 "" H 750 2750 50  0001 C CNN
-	1    750  2750
-	1    0    0    -1
-$EndComp
-Wire Wire Line
-	750  2750 750  2650
-Wire Wire Line
-	750  2650 850  2650
-Wire Wire Line
-	1150 2650 1250 2650
-Wire Wire Line
-	1250 2350 1250 2450
-Connection ~ 1250 2450
-Wire Wire Line
-	1250 2450 1350 2450
-$Comp
-L power:+5V #PWR0120
-U 1 1 5D397168
-P 1250 1950
-F 0 "#PWR0120" H 1250 1800 50  0001 C CNN
-F 1 "+5V" H 1265 2123 50  0000 C CNN
-F 2 "" H 1250 1950 50  0001 C CNN
-F 3 "" H 1250 1950 50  0001 C CNN
-	1    1250 1950
-	1    0    0    -1
-$EndComp
-Wire Wire Line
-	1250 1950 1250 2050
-Wire Wire Line
-	1250 2450 1250 2650
-Wire Wire Line
-	1250 2650 1350 2650
-Connection ~ 1250 2650
-$Comp
-L power:GND #PWR0121
-U 1 1 5D39BF62
-P 1850 2750
-F 0 "#PWR0121" H 1850 2500 50  0001 C CNN
-F 1 "GND" H 1855 2577 50  0000 C CNN
-F 2 "" H 1850 2750 50  0001 C CNN
-F 3 "" H 1850 2750 50  0001 C CNN
-	1    1850 2750
-	1    0    0    -1
-$EndComp
-Wire Wire Line
-	1850 2750 1850 2650
-Wire Wire Line
-	1850 2650 1750 2650
-Wire Wire Line
-	1750 2450 1850 2450
-Wire Wire Line
-	1850 2450 1850 2650
-Connection ~ 1850 2650
-Text Label 1250 2450 2    50   ~ 0
-BTN
 Text Label 3400 3100 0    50   ~ 0
 UP
@@
 P 4600 3200
 F 0 "J1" H 4628 3226 50  0000 L CNN
-F 1 "Conn_01x01_Female" H 4628 3135 50  0000 L CNN
+F 1 "5V" H 4628 3135 50  0000 L CNN
 F 2 "TestPoint:TestPoint_THTPad_D1.0mm_Drill0.5mm" H 4600 3200 50  0001 C CNN
 F 3 "~" H 4600 3200 50  0001 C CNN
@@
 L power:GND #PWR0116
 U 1 1 5D38663C
-P 4300 4200
-F 0 "#PWR0116" H 4300 3950 50  0001 C CNN
-F 1 "GND" H 4305 4027 50  0000 C CNN
-F 2 "" H 4300 4200 50  0001 C CNN
-F 3 "" H 4300 4200 50  0001 C CNN
-	1    4300 4200
+P 4300 4050
+F 0 "#PWR0116" H 4300 3800 50  0001 C CNN
+F 1 "GND" H 4305 3877 50  0000 C CNN
+F 2 "" H 4300 4050 50  0001 C CNN
+F 3 "" H 4300 4050 50  0001 C CNN
+	1    4300 4050
 	1    0    0    -1
 $EndComp
@@
 L Connector:Conn_01x01_Female J7
 U 1 1 5D386BCE
-P 4600 4100
-F 0 "J7" H 4628 4126 50  0000 L CNN
-F 1 "Conn_01x01_Female" H 4628 4035 50  0000 L CNN
-F 2 "TestPoint:TestPoint_THTPad_D1.0mm_Drill0.5mm" H 4600 4100 50  0001 C CNN
-F 3 "~" H 4600 4100 50  0001 C CNN
-	1    4600 4100
-	1    0    0    -1
-$EndComp
-Wire Wire Line
-	4300 4200 4300 4100
-Wire Wire Line
-	4300 4100 4400 4100
+P 4600 3950
+F 0 "J7" H 4628 3976 50  0000 L CNN
+F 1 "GND" H 4628 3885 50  0000 L CNN
+F 2 "TestPoint:TestPoint_THTPad_D1.0mm_Drill0.5mm" H 4600 3950 50  0001 C CNN
+F 3 "~" H 4600 3950 50  0001 C CNN
+	1    4600 3950
+	1    0    0    -1
+$EndComp
+Wire Wire Line
+	4300 4050 4300 3950
+Wire Wire Line
+	4300 3950 4400 3950
 $Comp
 L Connector:Conn_01x01_Female J2
@@
 P 4600 3350
 F 0 "J2" H 4628 3376 50  0000 L CNN
-F 1 "Conn_01x01_Female" H 4628 3285 50  0000 L CNN
+F 1 "UP" H 4628 3285 50  0000 L CNN
 F 2 "TestPoint:TestPoint_THTPad_D1.0mm_Drill0.5mm" H 4600 3350 50  0001 C CNN
 F 3 "~" H 4600 3350 50  0001 C CNN
@@
 P 4600 3500
 F 0 "J3" H 4628 3526 50  0000 L CNN
-F 1 "Conn_01x01_Female" H 4628 3435 50  0000 L CNN
+F 1 "R" H 4628 3435 50  0000 L CNN
 F 2 "TestPoint:TestPoint_THTPad_D1.0mm_Drill0.5mm" H 4600 3500 50  0001 C CNN
 F 3 "~" H 4600 3500 50  0001 C CNN
@@
 P 4600 3650
 F 0 "J4" H 4628 3676 50  0000 L CNN
-F 1 "Conn_01x01_Female" H 4628 3585 50  0000 L CNN
+F 1 "D" H 4628 3585 50  0000 L CNN
 F 2 "TestPoint:TestPoint_THTPad_D1.0mm_Drill0.5mm" H 4600 3650 50  0001 C CNN
 F 3 "~" H 4600 3650 50  0001 C CNN
@@
 P 4600 3800
 F 0 "J5" H 4628 3826 50  0000 L CNN
-F 1 "Conn_01x01_Female" H 4628 3735 50  0000 L CNN
+F 1 "L" H 4628 3735 50  0000 L CNN
 F 2 "TestPoint:TestPoint_THTPad_D1.0mm_Drill0.5mm" H 4600 3800 50  0001 C CNN
 F 3 "~" H 4600 3800 50  0001 C CNN
 	1    4600 3800
-	1    0    0    -1
-$EndComp
-$Comp
-L Connector:Conn_01x01_Female J6
-U 1 1 5D38DA7A
-P 4600 3950
-F 0 "J6" H 4628 3976 50  0000 L CNN
-F 1 "Conn_01x01_Female" H 4628 3885 50  0000 L CNN
-F 2 "TestPoint:TestPoint_THTPad_D1.0mm_Drill0.5mm" H 4600 3950 50  0001 C CNN
-F 3 "~" H 4600 3950 50  0001 C CNN
-	1    4600 3950
 	1    0    0    -1
 $EndComp
@@
 Text Label 4400 3650 2    50   ~ 0
 DOWN
-Text Label 4400 3950 2    50   ~ 0
-BTN
 $EndSCHEMATC
