File: main.kicad_pcb (KiCad board)
At the start: 2 copper layers, 307.3 x 96.1 mm, 153 parts, among them J1 RJ45, J2 RJ45, J3 RJ45, J4 RJ45, J5 USB_C_Receptacle_USB2.0, J6 STLinkV3, M1 MountingHole_2.2mm_M2, M10 MountingHole_2.2mm_M2, M11 MountingHole_2.2mm_M2, M12 MountingHole_2.2mm_M2, M13 MountingHole_2.2mm_M2, M14 MountingHole_2.2mm_M2, M15 MountingHole_2.2mm_M2, M16 MountingHole_2.2mm_M2, M17 MountingHole_2.2mm_M2, M2 MountingHole_2.2mm_M2, M20 MountingHole_2.2mm_M, M3 MountingHole_2.2mm_M2, M4 MountingHole_2.2mm_M2, M5 MountingHole_2.2mm_M2, M6 MountingHole_2.2mm_M2, M7 MountingHole_2.2mm_M2, M8 MountingHole_2.2mm_M2, M9 MountingHole_2.2mm_M2, SW1 K11, SW10 K42, SW11 K52, SW12 K62, SW13 K13, SW14 K23, SW15 K33, SW16 K43, SW17 K53, SW18 K63, SW19 K14, SW2 K21, SW20 K24, SW21 K34, SW22 K44, SW23 RST, SW24 BOOT0, SW25 BOOT1, SW26 K54, SW29 K64, SW3 K31, SW30 K71, SW31 K81, SW32 K91, SW33 K101, SW34 K111, SW35 K121, SW36 K72, SW37 K82, SW38 K92, SW39 K102, SW4 K41, SW40 K112, SW41 K122, SW42 K73, SW43 K83, SW44 K93, SW45 K103, SW46 K113, SW47 K123, SW48 K74, SW49 K84, SW5 K51, SW50 K94, SW51 K104, SW52 K114, SW53 K124, SW6 K61, SW7 K12, SW8 K22, SW9 K32, U1 STM32F401RETx, U2 AP131-33, Y1 8MHz, Y2 32.768kHz

Commit message: complete ver
Parts:
- added D25: LINKUP, LED_SMD:LED_0603_1608Metric_Pad1.05x0.95mm_HandSolder, F.Cu at (350.5, 415.3)
- added D26: L0, LED_SMD:LED_0603_1608Metric_Pad1.05x0.95mm_HandSolder, F.Cu at (353.2, 476.4)
- added D27: L1, LED_SMD:LED_0603_1608Metric_Pad1.05x0.95mm_HandSolder, F.Cu at (353.2, 478.3)
- added D52: L2, LED_SMD:LED_0603_1608Metric_Pad1.05x0.95mm_HandSolder, F.Cu at (353.2, 480.2)
- added R10: 220ohm, Resistor_SMD:R_0402_1005Metric_Pad0.72x0.64mm_HandSolder, F.Cu at (350.0, 478.3)
- added R11: 220ohm, Resistor_SMD:R_0402_1005Metric_Pad0.72x0.64mm_HandSolder, F.Cu at (350.0, 480.2)
- added R8: 220ohm, Resistor_SMD:R_0402_1005Metric_Pad0.72x0.64mm_HandSolder, F.Cu at (350.5, 417.8)
- added R9: 220ohm, Resistor_SMD:R_0402_1005Metric_Pad0.72x0.64mm_HandSolder, F.Cu at (350.0, 476.4)
- J6: footprint Connector_PinHeader_1.27mm:PinHeader_2x07_P1.27mm_Vertical -> folivora:IDC-Header_2x07_P1.27mm_Vertical
- moved R1 25.7 mm to (363.6, 452.9), turned to 180 degrees
- moved SW23 21.0 mm to (358.1, 454.8), turned to 180 degrees
- moved J6 9.66 mm to (351.9, 473.5), turned to 90 degrees
- moved C18 6.75 mm to (374.0, 469.9), turned to 180 degrees
- moved C2 3.18 mm to (377.1, 470.5), turned to 0 degrees
- moved Y2 3.11 mm to (364.2, 457.7)
- moved C10 3.11 mm to (366.1, 457.1)
- moved C11 3.11 mm to (366.1, 459.6)
- moved C1 2.32 mm to (379.3, 469.4)
- moved C5 2.32 mm to (367.9, 457.3)
- moved U1 2.32 mm to (374.3, 462.4)
- moved C3 2.32 mm to (366.6, 464.3)
- moved C4 2.32 mm to (380.0, 456.7)
- moved R2 1.81 mm to (363.2, 461.6)
- moved C9 1.81 mm to (360.0, 466.1)
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Connections:
- U1 pad 14: (no net) -> /LAYER1
- U1 pad 15: (no net) -> /LAYER2
- U1 pad 34: /COL12 -> /COL9
- U1 pad 35: /COL11 -> /COL10
- U1 pad 36: /COL10 -> /COL11
- U1 pad 37: /COL9 -> /COL12
- U1 pad 8: (no net) -> /LINKUP
- U1 pad 9: (no net) -> /LAYER0
Routing:
- net /LINKUP: track 0.00 -> 57.1 mm, vias 0 -> 2
- net +3V3: track 110.3 -> 163.3 mm, vias 6 -> 9
- net /LAYER0: track 0.00 -> 24.0 mm, vias 0 -> 2
- net /LAYER2: track 0.00 -> 22.2 mm, vias 0 -> 2
- net /LAYER1: track 0.00 -> 21.3 mm, vias 0 -> 2
- net /D-: track 58.4 -> 77.9 mm
- net /D+: track 57.8 -> 77.2 mm
- net /BOOT1: track 48.4 -> 30.6 mm
- net /COL1: track 41.1 -> 28.6 mm, vias 2 -> 0
- net /COL10: track 133.3 -> 121.8 mm, vias 1 -> 0
- net /COL12: track 171.5 -> 181.9 mm, vias 1 -> 0
- net /RST: track 33.6 -> 42.4 mm, vias 1 -> 5
- net /JTMS: track 23.7 -> 32.3 mm, vias 1 -> 2
- net /ROW1: track 142.0 -> 149.1 mm
- net /COL11: track 148.4 -> 141.4 mm, vias 1 -> 0
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- added copper zone on B.Cu, net GND1

Commit message: adjust silks
Other:
- board text added: "BOOT0"
- board text added: "BOOT1"
- board text added: "COL"
- board text added: "Col"
- board text added: "Layer 0"
- board text added: "Layer 1"
- board text added: "Layer 2"
- board text added: "Link"
- board text added: "ROW"
- board text added: "Reset"
- board text added: "Row"
- board text added: "namachan10777"
